File: schematic_pcb/Bluetooth_Car_Controller.kicad_pcb (KiCad board)
At the start: 2 copper layers, 82 x 53 mm, 22 parts, among them J1 Conn_01x04_Pin, J2 USB_C_Receptacle_PowerOnly_6P, J3 Conn_01x04_Pin, SW1 Prev_Button, SW2 Play_Pause, SW3 Next_Button, SW4 PROG, SW5 RESET, U1 MIC5504-3.3YM5, U2 ESP32-WROOM-32E

Commit message: Finish schematic and final code
Parts:
- moved J1 13.2 mm to (122.9, 112.7)
- moved C2 5.52 mm to (126.5, 117.0)
Routing:
- net +5V: track 123.4 -> 135.2 mm, vias 1 -> 2
- net /SCL: track 22.2 -> 15.9 mm
- net /SDA: track 21.4 -> 15.3 mm
- net GND: track 380.3 -> 385.5 mm, vias 4 -> 3
- net Net-(U2-EN): track 58.9 -> 59.0 mm, vias 3 -> 1
