File: schematic_pcb/Bluetooth_Car_Controller.kicad_sch (KiCad schematic)
At the start: 22 parts, among them J1 Conn_01x04_Pin, J2 USB_C_Receptacle_PowerOnly_6P, J3 Conn_01x04_Pin, SW1 Prev_Button, SW2 Play_Pause, SW3 Next_Button, SW4 PROG, SW5 RESET, U1 MIC5504-3.3YM5, U2 ESP32-WROOM-32E

Commit message: Finalize code and schematic
Other:
- note added: "Connected incorrectly, should be between switch + resistor"
- note added: "EN pin should be connected to 3.3V with pull down resistor"
Changed lines of the file:
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@@
+		)
+	)
+	(text "Connected incorrectly, should be between switch + resistor"
+		(exclude_from_sim no)
+		(at 247.65 75.692 0)
+		(effects
+			(font
+				(size 1.27 1.27)
+			)
 		)
 	)
@@
 		(effects
 			(font
+				(size 1.27 1.27)
+			)
+		)
+	)
+	(text "EN pin should be connected to 3.3V with pull down resistor"
+		(exclude_from_sim no)
+		(at 73.152 69.088 0)
+		(effects
+			(font
